File: pick-to-light.sch (KiCad schematic (older format))
At the start: 21 parts, among them P1 CONN_02X03, P2 CONN_02X03, Q1 BC849, Q2 BC849, SW1 SW_PUSH, SW2 SW_PUSH

Commit message: Started to hack the node design for custom ATMEGA168P circuit
Parts:
- added IC?: ATMEGA168PA-A, TQFP32, symbol ATMEGA168PA-A
Connections:
- wire segments 119 -> 75
- no-connect marks 10 -> 3
Other:
- moved on the sheet: P1, P2

Commit message: Fleshing out the circuit, need to check against pro mini reference and actual board design
Parts:
- removed ARD1: Arduino_Pro_Mini_Board, PTL-footprints:ArduinoProMini, symbol Arduino_Pro_Mini_Board
- added C? (x2): C, symbol C
- added C? (x3): 0.1uF, symbol C
- added R?: 10k, symbol R
- added SW?: reset, symbol SW_PUSH
- added Y?: Crystal, symbol Crystal
- R10, R11: value 10K -> 10k
Connections:
- net labels added: A3, A4, A5, RESET, RX1, TX0, XTAL1, XTAL2
- wire segments 75 -> 186
- no-connect marks 3 -> 0
Other:
- moved on the sheet: IC?, P1, P2

Commit message: Added pdf printout for reference on this commit
Connections:
- net labels added: RAW
- wire segments 186 -> 187
Other:
- note added: "Need to put power supply circuit here."
Changed lines of the file:
@@
 L GND #PWR?
 U 1 1 565FF150
-P 10850 7750
-F 0 "#PWR?" H 10850 7500 50  0001 C CNN
-F 1 "GND" H 10850 7600 50  0000 C CNN
-F 2 "" H 10850 7750 60  0000 C CNN
-F 3 "" H 10850 7750 60  0000 C CNN
-	1    10850 7750
-	1    0    0    -1
-$EndComp
-$Comp
-L VCC #PWR?
-U 1 1 56600626
-P 11100 8550
-F 0 "#PWR?" H 11100 8400 50  0001 C CNN
-F 1 "VCC" H 11100 8700 50  0000 C CNN
-F 2 "" H 11100 8550 60  0000 C CNN
-F 3 "" H 11100 8550 60  0000 C CNN
-	1    11100 8550
+P 10700 7750
+F 0 "#PWR?" H 10700 7500 50  0001 C CNN
+F 1 "GND" H 10700 7600 50  0000 C CNN
+F 2 "" H 10700 7750 60  0000 C CNN
+F 3 "" H 10700 7750 60  0000 C CNN
+	1    10700 7750
 	1    0    0    -1
 $EndComp
@@
 	4800 7100 6750 7100
 Wire Wire Line
-	10850 7550 10850 7750
-Wire Wire Line
-	11050 7550 11050 8000
-Wire Wire Line
-	11050 8000 11250 8000
-Wire Wire Line
-	11100 8600 11100 8550
+	10850 7650 10700 7650
+Wire Wire Line
+	11050 7550 11050 8200
+Wire Wire Line
+	11050 8200 10400 8200
 Wire Wire Line
 	4800 6900 6400 6900
@@
 	4800 7450 6350 7450
 Wire Wire Line
-	10400 7600 10950 7600
-Wire Wire Line
-	10950 7600 10950 7550
+	10400 8050 10950 8050
+Wire Wire Line
+	10950 8050 10950 7550
 Connection ~ 2500 8050
 $Comp
@@
 	4800 6350 4950 6350
 Wire Wire Line
-	14050 2650 13750 2650
-Wire Wire Line
-	13750 2650 13450 2650
+	13450 2650 13750 2650
+Wire Wire Line
+	13750 2650 14050 2650
 Wire Wire Line
 	13750 2650 13750 2600
@@
 	4800 6450 4850 6450
 Wire Wire Line
-	14050 2250 13750 2250
-Wire Wire Line
-	13750 2250 13450 2250
+	13450 2250 13750 2250
+Wire Wire Line
+	13750 2250 14050 2250
 Wire Wire Line
 	13750 2250 13750 2300
@@
 $EndComp
 Wire Wire Line
-	14750 2950 14750 2650
+	14750 2650 14750 2950
 Wire Wire Line
 	14500 2250 14350 2250
 Wire Wire Line
-	14750 2650 14500 2650
-Wire Wire Line
-	14500 2650 14350 2650
+	14350 2650 14500 2650
+Wire Wire Line
+	14500 2650 14750 2650
 Wire Wire Line
 	14500 2650 14500 2250
@@
 Wire Wire Line
 	10950 6750 10950 7050
-Text GLabel 10400 7600 0    60   Input ~ 0
+Text GLabel 10400 8050 0    60   Input ~ 0
 RESET
 Text GLabel 10400 6600 0    60   BiDi ~ 0
@@
 XTAL2
 Connection ~ 14500 2650
+Text GLabel 3050 9550 0    60   Input ~ 0
+RAW
+Text GLabel 10400 8200 0    60   Input ~ 0
+RAW
+Wire Wire Line
+	10850 7650 10850 7550
+Wire Wire Line
+	10700 7650 10700 7750
+Text Notes 5150 9600 2    60   ~ 0
+Need to put power supply circuit here.
 $EndSCHEMATC

Commit message: Added power supply circuit to schematic
Parts:
- added C3: 10uF, symbol C
- added C4: 22uF, symbol C
- added C5: 0.1uF, symbol C
- added R13, R14: 22k, symbol R
- added U1: LD1117S33TR, SOT-223, symbol LD1117S33TR
- R1, R2, R3, R4, R5, R6, R7, R8: value 510 -> 110
- gave numbers to parts that had none: 9
Connections:
- wire segments 187 -> 180
- no-connect marks 0 -> 5
Other:
- note removed: "Need to put power supply circuit here."

Commit message: Completed first itteration of layout. Needs spacing out and rerouting.
Parts:
- removed SW3: reset, symbol SW_PUSH
- added R16: 0, Capacitors_SMD:C_0603_HandSoldering, symbol R
- C1, C2, C3, C4, C5, C7, C8: footprint (none) -> Capacitors_SMD:C_0805
- C6: footprint (none) -> Capacitors_SMD:C_0805_HandSoldering
- IC1: footprint TQFP32 -> PTL-footprints:LQFP-32_5x5mm_Pitch0.5mm
- P1: footprint PTL-footprints:2x3-male-pin-header-smd -> PTL-footprints:2x3-male-pin-header-smd-board-edge
- P2: footprint PTL-footprints:2x3-male-pin-header-smd -> PTL-footprints:prog_smd_pads
- R1, R10, R11, R12, R2, R3, R4, R5, R6, R7, R8, R9: footprint Resistors_SMD:R_0805_HandSoldering -> Resistors_SMD:R_0805
- R13, R14, R15: footprint (none) -> Resistors_SMD:R_0805
- U1: footprint SOT-223 -> TO_SOT_Packages_SMD:SOT89-3_Housing
- Y1: footprint (none) -> Crystals:Crystal_HC49-U_Vertical
Connections:
- wire segments 180 -> 181

Commit message: Finished second round of layout.
Parts:
- removed C1: 0.1uF, Capacitors_SMD:C_0805, symbol C
- Q1, Q2: footprint TO_SOT_Packages_SMD:SOT-23_Handsoldering -> TO_SOT_Packages_SMD:SOT-23
Connections:
- wire segments 181 -> 179
Changed lines of the file:
@@
 F 0 "Q1" H 9500 3875 50  0000 L CNN
 F 1 "BC849" H 9500 3800 50  0000 L CNN
-F 2 "TO_SOT_Packages_SMD:SOT-23_Handsoldering" H 9500 3725 50  0001 L CIN
+F 2 "TO_SOT_Packages_SMD:SOT-23" H 9500 3725 50  0001 L CIN
 F 3 "" H 9300 3800 50  0000 L CNN
 	1    9300 3800
@@
 F 0 "Q2" H 11800 3875 50  0000 L CNN
 F 1 "BC849" H 11800 3800 50  0000 L CNN
-F 2 "TO_SOT_Packages_SMD:SOT-23_Handsoldering" H 11800 3725 50  0001 L CIN
+F 2 "TO_SOT_Packages_SMD:SOT-23" H 11800 3725 50  0001 L CIN
 F 3 "" H 11600 3800 50  0000 L CNN
 	1    11600 3800
@@
 Connection ~ 2500 5850
 $Comp
-L VCC #PWR011
-U 1 1 56623440
-P 1350 6450
-F 0 "#PWR011" H 1350 6300 50  0001 C CNN
-F 1 "VCC" H 1350 6600 50  0000 C CNN
-F 2 "" H 1350 6450 60  0000 C CNN
-F 3 "" H 1350 6450 60  0000 C CNN
-	1    1350 6450
-	1    0    0    -1
-$EndComp
-$Comp
-L GND #PWR012
-U 1 1 5662350B
-P 1350 6900
-F 0 "#PWR012" H 1350 6650 50  0001 C CNN
-F 1 "GND" H 1350 6750 50  0000 C CNN
-F 2 "" H 1350 6900 60  0000 C CNN
-F 3 "" H 1350 6900 60  0000 C CNN
-	1    1350 6900
-	1    0    0    -1
-$EndComp
-$Comp
-L C C1
-U 1 1 56623626
-P 1350 6650
-F 0 "C1" H 1375 6750 50  0000 L CNN
-F 1 "0.1uF" H 1375 6550 50  0000 L CNN
-F 2 "Capacitors_SMD:C_0805" H 1388 6500 30  0001 C CNN
-F 3 "" H 1350 6650 60  0000 C CNN
-	1    1350 6650
-	1    0    0    -1
-$EndComp
-Wire Wire Line
-	1350 6900 1350 6800
-Wire Wire Line
-	1350 6450 1350 6500
-$Comp
-L GND #PWR013
+L GND #PWR011
 U 1 1 56624C06
 P 2100 6900
-F 0 "#PWR013" H 2100 6650 50  0001 C CNN
+F 0 "#PWR011" H 2100 6650 50  0001 C CNN
 F 1 "GND" H 2100 6750 50  0000 C CNN
 F 2 "" H 2100 6900 60  0000 C CNN
@@
 $EndComp
 $Comp
-L VCC #PWR014
+L VCC #PWR012
 U 1 1 56627364
 P 14150 6300
-F 0 "#PWR014" H 14150 6150 50  0001 C CNN
+F 0 "#PWR012" H 14150 6150 50  0001 C CNN
 F 1 "VCC" H 14150 6450 50  0000 C CNN
 F 2 "" H 14150 6300 60  0000 C CNN
@@
 	14150 6700 14150 7150
 $Comp
-L GND #PWR015
+L GND #PWR013
 U 1 1 566275F1
 P 14800 7350
-F 0 "#PWR015" H 14800 7100 50  0001 C CNN
+F 0 "#PWR013" H 14800 7100 50  0001 C CNN
 F 1 "GND" H 14800 7200 50  0000 C CNN
 F 2 "" H 14800 7350 60  0000 C CNN
@@
 	7300 9450 8000 9450
 $Comp
-L VCC #PWR016
+L VCC #PWR014
 U 1 1 5666D179
 P 9650 9300
-F 0 "#PWR016" H 9650 9150 50  0001 C CNN
+F 0 "#PWR014" H 9650 9150 50  0001 C CNN
 F 1 "VCC" H 9650 9450 50  0000 C CNN
 F 2 "" H 9650 9300 60  0000 C CNN
@@
 	9650 9450 9650 9300
 $Comp
-L GND #PWR017
+L GND #PWR015
 U 1 1 5666DB60
 P 8400 10300
-F 0 "#PWR017" H 8400 10050 50  0001 C CNN
+F 0 "#PWR015" H 8400 10050 50  0001 C CNN
 F 1 "GND" H 8400 10150 50  0000 C CNN
 F 2 "" H 8400 10300 60  0000 C CNN
@@
 Connection ~ 7450 7100
 $Comp
-L VCC #PWR018
+L VCC #PWR016
 U 1 1 5667583B
 P 7350 6500
-F 0 "#PWR018" H 7350 6350 50  0001 C CNN
+F 0 "#PWR016" H 7350 6350 50  0001 C CNN
 F 1 "VCC" H 7350 6650 50  0000 C CNN
 F 2 "" H 7350 6500 60  0000 C CNN
